File: Turbidometer.kicad_pcb (KiCad board)
At the start: 2 copper layers, 36 x 36 mm, 16 parts, among them IC1 BH1730FVC-TR, IC2 NLSX4373DR2G, J1 Conn_01x04, J2 Conn_01x04, U1 LP2985-3.0

Commit message: Adding useful silk
Other:
- board text added: "3V3"
- board text added: "GND"
- board text added: "SCL"
- board text added: "SDA"
- board text added: "Vin"
Changed lines of the file:
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@@
     (property "ki_keywords" "connector")
     (attr smd)
-    (fp_text reference "J1" (at 0.5 -3.98) (layer "F.SilkS")
+    (fp_text reference "J1" (at 4.25 -1.25) (layer "F.SilkS")
         (effects (font (size 1 1) (thickness 0.15)))
     )
@@
     (property "ki_keywords" "mounting hole")
     (attr exclude_from_pos_files)
-    (fp_text reference "H2" (at 0 -3.75) (layer "F.SilkS")
+    (fp_text reference "H2" (at 0 -3.75) (layer "F.SilkS") hide
         (effects (font (size 1 1) (thickness 0.15)))
     )
@@
     (property "ki_description" "2-Bit 20 Mb/s Dual-Supply Level Translator")
     (attr smd)
-    (fp_text reference "IC2" (at -2.4 3.75) (layer "F.SilkS")
+    (fp_text reference "IC2" (at -5.15 0.5) (layer "F.SilkS")
         (effects (font (size 1 1) (thickness 0.15)))
     )
@@
     (property "ki_keywords" "mounting hole")
     (attr exclude_from_pos_files)
-    (fp_text reference "H1" (at 0 -3.75) (layer "F.SilkS")
+    (fp_text reference "H1" (at 0 -3.75) (layer "F.SilkS") hide
         (effects (font (size 1 1) (thickness 0.15)))
     )
@@
     (property "ki_keywords" "mounting hole")
     (attr exclude_from_pos_files)
-    (fp_text reference "H4" (at 0 -3.75 180) (layer "F.SilkS")
+    (fp_text reference "H4" (at 0 -3.75 180) (layer "F.SilkS") hide
         (effects (font (size 1 1) (thickness 0.15)))
     )
@@
     (property "ki_keywords" "mounting hole")
     (attr exclude_from_pos_files)
-    (fp_text reference "H3" (at 0 -3.75 180) (layer "F.SilkS")
+    (fp_text reference "H3" (at 0 -3.75 180) (layer "F.SilkS") hide
         (effects (font (size 1 1) (thickness 0.15)))
     )
@@
     (property "ki_keywords" "connector")
     (attr through_hole)
-    (fp_text reference "J2" (at 3.75 -3.55) (layer "F.SilkS")
+    (fp_text reference "J2" (at -4 -2.25) (layer "F.SilkS")
         (effects (font (size 1 1) (thickness 0.15)))
     )
@@
   (gr_arc (start 123 77.5) (mid 122.12132 79.62132) (end 120 80.5)
     (stroke (width 0.1) (type default)) (layer "Edge.Cuts"))
+  (gr_text "Vin" (at 109.5 54.5 270) (layer "B.SilkS")
+    (effects (font (size 1 1) (thickness 0.15)) (justify left bottom mirror))
+  )
+  (gr_text "SDA" (at 107 54.5 -90) (layer "B.SilkS")
+    (effects (font (size 1 1) (thickness 0.15)) (justify left bottom mirror))
+  )
+  (gr_text "GND" (at 112 54.75 -90) (layer "B.SilkS")
+    (effects (font (size 1 1) (thickness 0.15)) (justify left bottom mirror))
+  )
+  (gr_text "SCL" (at 104.5 54.5 -90) (layer "B.SilkS")
+    (effects (font (size 1 1) (thickness 0.15)) (justify left bottom mirror))
+  )
+  (gr_text "Vin" (at 110.75 54.5 90) (layer "F.SilkS")
+    (effects (font (size 1 1) (thickness 0.15)) (justify left bottom))
+  )
+  (gr_text "SDA" (at 108.25 54.5 90) (layer "F.SilkS")
+    (effects (font (size 1 1) (thickness 0.15)) (justify left bottom))
+  )
+  (gr_text "SDA" (at 98 54 90) (layer "F.SilkS")
+    (effects (font (size 0.5 0.5) (thickness 0.1)) (justify left bottom))
+  )
+  (gr_text "GND" (at 113.25 54.75 90) (layer "F.SilkS")
+    (effects (font (size 1 1) (thickness 0.15)) (justify left bottom))
+  )
+  (gr_text "3V3" (at 99 54 90) (layer "F.SilkS")
+    (effects (font (size 0.5 0.5) (thickness 0.1) bold) (justify left bottom))
+  )
+  (gr_text "SCL" (at 105.75 54.5 90) (layer "F.SilkS")
+    (effects (font (size 1 1) (thickness 0.15)) (justify left bottom))
+  )
+  (gr_text "SCL" (at 97 54 90) (layer "F.SilkS")
+    (effects (font (size 0.5 0.5) (thickness 0.1) bold) (justify left bottom))
+  )
+  (gr_text "GND" (at 100 54 90) (layer "F.SilkS")
+    (effects (font (size 0.5 0.5) (thickness 0.1) bold) (justify left bottom))
+  )
   (dimension (type aligned) (layer "Dwgs.User")
     (pts (xy 87 77.5) (xy 123 77.5))

Commit message: adding teardrops, fixing silk
Routing:
- net GND: vias 45 -> 52
